File: CorruptCore.brd (EAGLE design)
At the start: 100 x 100 mm, 89 parts, among them IC1 MEGA8-P, K1 DTS-3, K10 DTS-3, K11 DTS-3, K12 DTS-3, K13 DTS-3, K14 DTS-3, K15 DTS-3, K16 DTS-3, K2 DTS-3, K3 DTS-3, K4 DTS-3, K5 DTS-3, K6 DTS-3, K7 DTS-3, K8 DTS-3, K9 DTS-3, Y1 16MHz

Commit message: -added a PNG of the schematic -small amounts of schematic cleaning
Connections:
- net GND: now also U$5.9
Changed lines of the file:
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@@
 <contactref element="Q3" pad="2"/>
 <contactref element="Q4" pad="2"/>
+<contactref element="U$5" pad="9"/>
 <wire x1="-152" y1="-1329" x2="-152" y2="-1355" width="0" layer="19" extent="1-1"/>
 <wire x1="-152" y1="-1433" x2="-152" y2="-1355" width="0" layer="19" extent="1-1"/>
@@
 <wire x1="-46.64" y1="-94.61" x2="-152" y2="-1355" width="0" layer="19" extent="1-1"/>
 <wire x1="-25.77" y1="-86.99" x2="-46.64" y2="-94.61" width="0" layer="19" extent="1-1"/>
-<wire x1="-15.61" y1="-94.61" x2="-25.77" y2="-86.99" width="0" layer="19" extent="1-1"/>
+<wire x1="-15.61" y1="-86.99" x2="-25.77" y2="-86.99" width="0" layer="19" extent="1-1"/>
+<wire x1="-15.61" y1="-94.61" x2="-15.61" y2="-86.99" width="0" layer="19" extent="1-1"/>
 <wire x1="-30.48" y1="2.54" x2="-25.77" y2="-86.99" width="0" layer="19" extent="1-1"/>
 <wire x1="-33.02" y1="10.16" x2="-30.48" y2="2.54" width="0" layer="19" extent="1-1"/>
