File: corrupt_core_eagle_files/CorruptCore.brd (EAGLE design)
At the start: 100 x 100 mm, 81 parts, among them K1 DTS-3, K10 DTS-3, K11 DTS-3, K12 DTS-3, K13 DTS-3, K14 DTS-3, K15 DTS-3, K16 DTS-3, K2 DTS-3, K3 DTS-3, K4 DTS-3, K5 DTS-3, K6 DTS-3, K7 DTS-3, K8 DTS-3, K9 DTS-3, U1 MEGA8-P, U2 SNX4HC595SOIC16, U3 SNX4HC595SOIC16, U4 SNX4HC595SOIC16, U5 ULN2803ASOIC18, U6 ULN2803ASOIC18, U7 ULN2803ASOIC18, Y1 16MHz

Commit message: -more board changes
Parts:
- moved T1 66.5 mm to (70.0, 40.0)
- moved T2 66.5 mm to (64.0, 40.0)
- moved T3 66.5 mm to (58.0, 40.0)
- moved T4 66.5 mm to (52.0, 40.0)
- moved 5V@PROG 45.4 mm to (-36.0, 36.0)
- moved R3 29.6 mm to (5.00, 16.0), flipped to the bottom, turned to 90 degrees
- moved R2 23.2 mm to (2.00, 16.0), flipped to the bottom, turned to 90 degrees
- moved U6 8.59 mm to (24.0, 45.0)
- moved U5 8.30 mm to (10.0, 45.0)
- moved U7 8.29 mm to (38.0, 45.0)
- moved U4 7.94 mm to (37.0, 34.0)
- moved U3 7.55 mm to (24.0, 34.0)
- moved U2 7.27 mm to (11.0, 34.0)
- moved C1 3.16 mm to (34.0, 8.00), flipped to the bottom
- moved C2 3.16 mm to (28.0, 8.00), flipped to the bottom
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